File: haptic-keyboard/haptic-keyboard/keyboard.kicad_sch (KiCad schematic)
At the start: 111 parts, among them SW3 RotaryEncoder

Commit message: Added the initial schematic for it.
Parts:
- removed D1, D10, D100, D101, D102, D103, D104, D11, D12, D13, D14, D15, D16, D17, D18, D19, D2, D20, D21, D22, D23, D24, D25, D26, D27, D28, D29, D3, D30, D31, D32, D33, D34, D35, D36, D37, D38, D39, D4, D40, D41, D42, D43, D44, D45, D46, D47, D48, D49, D5, D50, D51, D52, D53, D54, D55, D56, D57, D58, D59, D6, D60, D61, D62, D63, D64, D65, D66, D67, D68, D69, D7, D70, D71, D72, D73, D74, D75, D76, D77, D78, D79, D8, D80, D81, D82, D83, D84, D85, D86, D87, D88, D89, D9, D90, D91, D92, D93, D94, D95, D96, D97, D98, D99: 1N4148W, Diode_SMD:D_SOD-123, symbol Diode:1N4148W
- removed D105, D106, D107, D108, D109, D110: WS2812B, LED_SMD:LED_WS2812B_PLCC4_5.0x5.0mm_P3.2mm, symbol LED:WS2812B
- removed SW3: RotaryEncoder, symbol Device:RotaryEncoder

Commit message: Finished Matrix Only!
Parts:
- added D10, D11, D12, D13, D14, D15, D16, D17, D18, D19, D2, D20, D21, D22, D23, D24, D25, D26, D27, D28, D29, D3, D30, D31, D32, D33, D34, D35, D36, D37, D38, D39, D4, D40, D41, D42, D43, D45, D46, D47, D48, D49, D5, D50, D51, D52, D53, D54, D55, D56, D57, D59, D6, D60, D61, D62, D63, D64, D68, D7, D72, D73, D74, D75, D76, D8, D9: D, symbol Device:D
- added SW10, SW11, SW12, SW13, SW14, SW15, SW16, SW17, SW18, SW19, SW2, SW20, SW21, SW22, SW23, SW24, SW25, SW26, SW27, SW28, SW29, SW3, SW30, SW31, SW32, SW33, SW34, SW35, SW36, SW37, SW38, SW39, SW4, SW40, SW41, SW42, SW43, SW45, SW46, SW47, SW48, SW49, SW5, SW50, SW51, SW52, SW53, SW54, SW55, SW56, SW57, SW59, SW6, SW60, SW61, SW62, SW63, SW64, SW68, SW7, SW72, SW73, SW74, SW75, SW76, SW8, SW9: SW_Push, symbol Switch:SW_Push
Connections:
- new net: D75.2 (A), SW75.1
- new net: D24.2 (A), SW24.1
- new net: D2.2 (A), SW2.1
- new net: D26.2 (A), SW26.1
- new net: D62.2 (A), SW62.1
- new net: D7.2 (A), SW7.1
- new net: D74.2 (A), SW74.1
- new net: D47.2 (A), SW47.1
- new net: D53.2 (A), SW53.1
- new net: D68.2 (A), SW68.1
- new net: D46.2 (A), SW46.1
- new net: D8.2 (A), SW8.1
- new net: D31.2 (A), SW31.1
- new net: D56.2 (A), SW56.1
- new net: D48.2 (A), SW48.1
- new net: D54.2 (A), SW54.1
- new net: D16.2 (A), SW16.1
- new net: D32.2 (A), SW32.1
- new net: D52.2 (A), SW52.1
- new net: D23.2 (A), SW23.1
- new net: D9.2 (A), SW9.1
- new net: D63.2 (A), SW63.1
- new net: D33.2 (A), SW33.1
- new net: D18.2 (A), SW18.1
- new net: D64.2 (A), SW64.1
- new net: D43.2 (A), SW43.1
- new net: D41.2 (A), SW41.1
- new net: D59.2 (A), SW59.1
- new net: D29.2 (A), SW29.1
- new net: D34.2 (A), SW34.1
- new net: D76.2 (A), SW76.1
- new net: D61.2 (A), SW61.1
- new net: D17.2 (A), SW17.1
- new net: D42.2 (A), SW42.1
- new net: D72.2 (A), SW72.1
- new net: D5.2 (A), SW5.1
- new net: D37.2 (A), SW37.1
- new net: D10.2 (A), SW10.1
- new net: D39.2 (A), SW39.1
- new net: D45.2 (A), SW45.1
- new net: D36.2 (A), SW36.1
- new net: D51.2 (A), SW51.1
- new net: D49.2 (A), SW49.1
- new net: D55.2 (A), SW55.1
- new net: D30.2 (A), SW30.1
- new net: D13.2 (A), SW13.1
- new net: D22.2 (A), SW22.1
- new net: D15.2 (A), SW15.1
- new net: D20.2 (A), SW20.1
- new net: D4.2 (A), SW4.1
- new net: D73.2 (A), SW73.1
- new net: D35.2 (A), SW35.1
- new net: D21.2 (A), SW21.1
- new net: D40.2 (A), SW40.1
- new net: D19.2 (A), SW19.1
- new net: D27.2 (A), SW27.1
- new net: D57.2 (A), SW57.1
- new net: D60.2 (A), SW60.1
- new net: D6.2 (A), SW6.1
- new net: D14.2 (A), SW14.1
- new net: D50.2 (A), SW50.1
- new net: D28.2 (A), SW28.1
- new net: D3.2 (A), SW3.1
- new net: D25.2 (A), SW25.1
- new net: D11.2 (A), SW11.1
- new net: D12.2 (A), SW12.1
- new net: D38.2 (A), SW38.1
- new net col0: SW17.2, SW2.2, SW32.2, SW47.2, SW62.2
- new net col1: SW18.2, SW3.2, SW33.2, SW48.2, SW63.2
- new net col10: SW12.2, SW27.2, SW42.2, SW57.2, SW72.2
- new net col11: SW13.2, SW28.2, SW43.2, SW73.2
- new net col12: SW14.2, SW29.2, SW59.2, SW74.2
- new net col13: SW15.2, SW30.2, SW45.2, SW60.2, SW75.2
- new net col14: D10.1 (K), D11.1 (K), D12.1 (K), D13.1 (K), D14.1 (K), D15.1 (K), D16.1 (K), D2.1 (K), D3.1 (K), D4.1 (K), D5.1 (K), D6.1 (K), D7.1 (K), D8.1 (K), D9.1 (K), SW16.2, SW31.2, SW46.2, SW61.2, SW76.2
- new net col2: SW19.2, SW34.2, SW4.2, SW49.2, SW64.2
- new net col3: SW20.2, SW35.2, SW5.2, SW50.2
- new net col4: SW21.2, SW36.2, SW51.2, SW6.2
- new net col5: SW22.2, SW37.2, SW52.2, SW7.2
- new net col6: SW23.2, SW38.2, SW53.2, SW68.2, SW8.2
- new net col7: SW24.2, SW39.2, SW54.2, SW9.2
- new net col8: SW10.2, SW25.2, SW40.2, SW55.2
- new net col9: SW11.2, SW26.2, SW41.2, SW56.2
- new net row1: D17.1 (K), D18.1 (K), D19.1 (K), D20.1 (K), D21.1 (K), D22.1 (K), D23.1 (K), D24.1 (K), D25.1 (K), D26.1 (K), D27.1 (K), D28.1 (K), D29.1 (K), D30.1 (K), D31.1 (K)
- new net row2: D32.1 (K), D33.1 (K), D34.1 (K), D35.1 (K), D36.1 (K), D37.1 (K), D38.1 (K), D39.1 (K), D40.1 (K), D41.1 (K), D42.1 (K), D43.1 (K), D45.1 (K), D46.1 (K)
- new net row3: D47.1 (K), D48.1 (K), D49.1 (K), D50.1 (K), D51.1 (K), D52.1 (K), D53.1 (K), D54.1 (K), D55.1 (K), D56.1 (K), D57.1 (K), D59.1 (K), D60.1 (K), D61.1 (K)
- new net row4: D62.1 (K), D63.1 (K), D64.1 (K), D68.1 (K), D72.1 (K), D73.1 (K), D74.1 (K), D75.1 (K), D76.1 (K)
